Commit message: v8

File: install/myrobot/share/myrobot/urdf/robot.urdf.xacro (robot description, xacro)
@@ -1,65 +1 @@
-<?xml version="1.0"?>
-<robot xmlns:xacro="http://www.ros.org/wiki/xacro" name="myrobot">
-  <link name="base_link">
-    <visual>
-      <geometry>
-        <box size="1 1 1"/>
-      </geometry>
-      <origin xyz="0 0 0.5" rpy="0 0 0"/>
-      <material name="grey">
-        <color rgba="0.5 0.5 0.5 1"/>
-      </material>
-    </visual>
-  </link>
-  <joint name="base_joint" type="fixed">
-    <parent link="base_link"/>
-    <child link="link_0"/>
-    <origin xyz="0 0 0" rpy="0 0 0"/>
-  </joint>
-  <xacro:macro name="link" params="name">
-    <link name="${name}">
-      <visual>
-        <geometry>
-          <box size="1 1 1"/>
-        </geometry>
-        <origin xyz="0 0 0.5" rpy="0 0 0"/>
-        <material name="grey">
-          <color rgba="0.5 0.5 0.5 1"/>
-        </material>
-      </visual>
-      <collision>
-        <geometry>
-          <box size="1 1 1"/>
-        </geometry>
-        <origin xyz="0 0 0.5" rpy="0 0 0"/>
-      </collision>
-      <inertial>
-        <mass value="0.5"/>
-        <inertia ixx="0.01" iyy="0.01" izz="0.01" ixy="0.0" ixz="0.0" iyz="0.0"/>
-        <origin xyz="0 0 0.5" rpy="0 0 0"/>
-      </inertial>
-    </link>
-  </xacro:macro>
-  <xacro:macro name="joint" params="name parent child xyz rpy axis lower upper">
-    <joint name="${name}" type="revolute">
-      <parent link="${parent}"/>
-      <child link="${child}"/>
-      <origin xyz="${xyz}" rpy="${rpy}"/>
-      <axis xyz="${axis}"/>
-      <limit lower="${lower}" upper="${upper}" effort="1.0" velocity="1.0"/>
-    </joint>
-  </xacro:macro>
-  <xacro:link name="link_0"/>
-  <xacro:link name="link_1"/>
-  <xacro:link name="link_2"/>
-  <xacro:link name="link_3"/>
-  <xacro:link name="link_4"/>
-  <xacro:link name="link_5"/>
-  <xacro:link name="link_6"/>
-  <xacro:joint name="joint_1" parent="link_0" child="link_1" xyz="0 1 0" rpy="-1.57 0 0" axis="0 0 1" lower="-3.14" upper="3.14"/>
-  <xacro:joint name="joint_2" parent="link_1" child="link_2" xyz="0 0 1" rpy="0 1.57 0" axis="0 0 1" lower="-0.86" upper="0.73"/>
-  <xacro:joint name="joint_3" parent="link_2" child="link_3" xyz="0 1 0" rpy="-1.57 0 0" axis="0 0 1" lower="-2.69" upper="2.31"/>
-  <xacro:joint name="joint_4" parent="link_3" child="link_4" xyz="0 0 1" rpy="1.57 0 0" axis="0 0 1" lower="-1.57" upper="1.45"/>
-  <xacro:joint name="joint_5" parent="link_4" child="link_5" xyz="0 1 0" rpy="-1.57 0 0" axis="0 0 1" lower="-3.14" upper="1.90"/>
-  <xacro:joint name="joint_6" parent="link_5" child="link_6" xyz="0 0 1" rpy="1.57 0 0" axis="0 0 1" lower="-0.57" upper="1.19"/>
-</robot>
+/home/pim0ubuntu/myrobot_ws/build/myrobot/urdf/robot.urdf.xacro

Commit message: v9

File: install/myrobot/share/myrobot/urdf/robot.urdf.xacro (robot description, xacro)
@@ -1 +1,65 @@
-/home/pim0ubuntu/myrobot_ws/build/myrobot/urdf/robot.urdf.xacro
+<?xml version="1.0"?>
+<robot xmlns:xacro="http://www.ros.org/wiki/xacro" name="myrobot">
+  <link name="base_link">
+    <visual>
+      <geometry>
+        <box size="1 1 1"/>
+      </geometry>
+      <origin xyz="0 0 0.5" rpy="0 0 0"/>
+      <material name="grey">
+        <color rgba="0.5 0.5 0.5 1"/>
+      </material>
+    </visual>
+  </link>
+  <joint name="base_joint" type="fixed">
+    <parent link="base_link"/>
+    <child link="link_0"/>
+    <origin xyz="0 0 0" rpy="0 0 0"/>
+  </joint>
+  <xacro:macro name="link" params="name">
+    <link name="${name}">
+      <visual>
+        <geometry>
+          <box size="1 1 1"/>
+        </geometry>
+        <origin xyz="0 0 0.5" rpy="0 0 0"/>
+        <material name="grey">
+          <color rgba="0.5 0.5 0.5 1"/>
+        </material>
+      </visual>
+      <collision>
+        <geometry>
+          <box size="1 1 1"/>
+        </geometry>
+        <origin xyz="0 0 0.5" rpy="0 0 0"/>
+      </collision>
+      <inertial>
+        <mass value="0.5"/>
+        <inertia ixx="0.01" iyy="0.01" izz="0.01" ixy="0.0" ixz="0.0" iyz="0.0"/>
+        <origin xyz="0 0 0.5" rpy="0 0 0"/>
+      </inertial>
+    </link>
+  </xacro:macro>
+  <xacro:macro name="joint" params="name parent child xyz rpy axis lower upper">
+    <joint name="${name}" type="revolute">
+      <parent link="${parent}"/>
+      <child link="${child}"/>
+      <origin xyz="${xyz}" rpy="${rpy}"/>
+      <axis xyz="${axis}"/>
+      <limit lower="${lower}" upper="${upper}" effort="1.0" velocity="1.0"/>
+    </joint>
+  </xacro:macro>
+  <xacro:link name="link_0"/>
+  <xacro:link name="link_1"/>
+  <xacro:link name="link_2"/>
+  <xacro:link name="link_3"/>
+  <xacro:link name="link_4"/>
+  <xacro:link name="link_5"/>
+  <xacro:link name="link_6"/>
+  <xacro:joint name="joint_1" parent="link_0" child="link_1" xyz="0 1 0" rpy="-1.57 0 0" axis="0 0 1" lower="-3.14" upper="3.14"/>
+  <xacro:joint name="joint_2" parent="link_1" child="link_2" xyz="0 0 1" rpy="0 1.57 0" axis="0 0 1" lower="-0.86" upper="0.73"/>
+  <xacro:joint name="joint_3" parent="link_2" child="link_3" xyz="0 1 0" rpy="-1.57 0 0" axis="0 0 1" lower="-2.69" upper="2.31"/>
+  <xacro:joint name="joint_4" parent="link_3" child="link_4" xyz="0 0 1" rpy="1.57 0 0" axis="0 0 1" lower="-1.57" upper="1.45"/>
+  <xacro:joint name="joint_5" parent="link_4" child="link_5" xyz="0 1 0" rpy="-1.57 0 0" axis="0 0 1" lower="-3.14" upper="1.90"/>
+  <xacro:joint name="joint_6" parent="link_5" child="link_6" xyz="0 0 1" rpy="1.57 0 0" axis="0 0 1" lower="-0.57" upper="1.19"/>
+</robot>
